File: hardware/ESP-v3locirap2rs_hardware/ESP32.kicad_sch (KiCad schematic)
At the start: 1 part, among them U1 ESP32-DEVKITC-32D

Commit message: pcb updates
Parts:
- U1: footprint digikey-footprints:MODULE_ESP32-DEVKITC-32D -> ESP-v3locirap2rs_footprints:MODULE_ESP32-DEVKITC-32D
Changed lines of the file:
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@@
 			)
 		)
-		(property "Footprint" "digikey-footprints:MODULE_ESP32-DEVKITC-32D"
+		(property "Footprint" "ESP-v3locirap2rs_footprints:MODULE_ESP32-DEVKITC-32D"
 			(at 135.89 100.33 0)
 			(effects

Commit message: schematic finalization
Connections:
- net 5V: now reaches U1.J2-19 (EXT_5V)
- net Pin 17: now reaches U1.J3-11 (IO17)
- net Pin 16: now reaches U1.J3-12 (IO16)
- net Pin 15: now reaches U1.J3-16 (IO15)
- net Pin 23: now reaches U1.J3-2 (IO23)
- net Pin 19: now reaches U1.J3-8 (IO19)
- net Pin 18: now reaches U1.J3-9 (IO18)
Changed lines of the file:
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@@
+		)
+	)
+	(hierarchical_label "Pin 23"
+		(shape output)
+		(at 156.21 80.01 0)
+		(fields_autoplaced yes)
+		(effects
+			(font
+				(size 1.27 1.27)
+			)
+			(justify left)
+		)
+	)
+	(hierarchical_label "Pin 17"
+		(shape output)
+		(at 156.21 102.87 0)
+		(fields_autoplaced yes)
+		(effects
+			(font
+				(size 1.27 1.27)
+			)
+			(justify left)
+		)
+	)
+	(hierarchical_label "Pin 19"
+		(shape output)
+		(at 156.21 95.25 0)
+		(fields_autoplaced yes)
+		(effects
+			(font
+				(size 1.27 1.27)
+			)
+			(justify left)
 		)
 	)
@@
 		(shape output)
 		(at 156.21 82.55 0)
+		(fields_autoplaced yes)
+		(effects
+			(font
+				(size 1.27 1.27)
+			)
+			(justify left)
+		)
+	)
+	(hierarchical_label "Pin 15"
+		(shape output)
+		(at 156.21 115.57 0)
 		(fields_autoplaced yes)
 		(effects
@@
 		)
 	)
+	(hierarchical_label "Pin 18"
+		(shape output)
+		(at 156.21 97.79 0)
+		(fields_autoplaced yes)
+		(effects
+			(font
+				(size 1.27 1.27)
+			)
+			(justify left)
+		)
+	)
+	(hierarchical_label "Pin 16"
+		(shape output)
+		(at 156.21 105.41 0)
+		(fields_autoplaced yes)
+		(effects
+			(font
+				(size 1.27 1.27)
+			)
+			(justify left)
+		)
+	)
 	(hierarchical_label "3.3V"
 		(shape output)
@@
 		(fields_autoplaced yes)
 		(effects
+			(font
+				(size 1.27 1.27)
+			)
+			(justify right)
+		)
+	)
+	(hierarchical_label "5V"
+		(shape input)
+		(at 115.57 123.19 180)
+		(fields_autoplaced yes)
+		(effects
