File: hardware/ESP-v3locirap2rs_hardware/LCD-Screen.kicad_sch (KiCad schematic)
At the start: 3 parts

Commit message: PCB completed
Parts:
- R1, R2: footprint (none) -> Resistor_SMD:R_0805_2012Metric
Changed lines of the file:
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@@
 			)
 		)
-		(property "Footprint" ""
+		(property "Footprint" "Resistor_SMD:R_0805_2012Metric"
 			(at 154.94 72.898 90)
 			(effects
@@
 			)
 		)
-		(property "Footprint" ""
+		(property "Footprint" "Resistor_SMD:R_0805_2012Metric"
 			(at 154.94 80.518 90)
 			(effects
