File: hardware/ESP-v3locirap2rs_hardware/ESP-v3locirap2rs_hardware.kicad_sch (KiCad schematic)
At the start: 0 parts

Commit message: schematic updates
Other:
- note added: "ESP32 Block"
Changed lines of the file:
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@@
+		)
+	)
+	(rectangle
+		(start 142.24 90.17)
+		(end 200.66 120.65)
+		(stroke
+			(width 0)
+			(type default)
+		)
+		(fill
+			(type none)
+		)
+	)
+	(text "ESP32 Block"
+		(exclude_from_sim no)
+		(at 149.098 89.154 0)
+		(effects
+			(font
+				(size 1.27 1.27)
+			)
 		)
 	)
